File: System Indicators/TSALv0.1/TSALv0.1.kicad_sch (KiCad schematic)
At the start: 3 parts, among them U1 LM311, U2 NA555P, U3 4N35

Commit message: Updated Schematic
Parts:
- added C1, C2: C, symbol Device:C
- added D1: D, symbol Device:D
- added Q1: 2N7002, Package_TO_SOT_SMD:SOT-23, symbol Transistor_FET:2N7002
- added R1, R10, R11, R12, R13, R14, R2, R3, R4, R5, R6, R7, R8, R9: R, symbol Device:R
- U?: renamed from U2; value NA555P -> NE555D; footprint Package_DIP:DIP-8_W7.62mm -> Package_SO:SOIC-8_3.9x4.9mm_P1.27mm; symbol Timer:NA555P -> Timer:NE555D
Connections:
- net at U3.1: now also R13.1
- net at U3.2: now also R12.2
- net at U3.4: now also Q1.1 (G), R14.1
- net VCC: now reaches U3.5
- net GND: now reaches U1.1 (GND)
- net GND: now also U1.4 (V-), C1.1, D1.2 (A), R6.1, R9.2
- net at U1.2 (+): now also C2.1, R10.2
- net at U1.3 (-): now also C2.2, R11.1
- net at U1.5 (BAL): now also U1.6 (STRB)
- net +12V: now reaches U1.8 (V+)
- net +12V: now also C1.2, R13.2, R7.1
- new net: R1.2, R2.1
- new net: R2.2, R3.2
- new net: D1.1 (K), R10.1, R12.1, R4.1, R5.2
- new net: R3.1, R4.2
- new net: R8.2, R9.1
- new net: R11.2, R7.2, R8.1
- new net: R5.1, R6.2
- new net -: Q1.2 (S), R14.2
- no-connect marks 0 -> 1
Other:
- note added: "Battery Connection Place holder"
- note added: "Isolated Power Supply & TSAL Light Interconnect"
- note added: "Refernce Voltage"
- note added: "Scale Main Voltage source"
- moved on the sheet: U?

Commit message: Finished Schemetic layout
Parts:
- added C3, C4, C5, C6: C, symbol Device:C
- added D2: D, symbol Device:D
- added D3: LED, symbol Device:LED
- added J1: Conn_01x06_Socket, symbol Connector:Conn_01x06_Socket
- added Q2: 2N7002, Package_TO_SOT_SMD:SOT-23, symbol Transistor_FET:2N7002
- added R15, R16, R17, R18, R19: R, symbol Device:R
Connections:
- net -: now also C3.1, D2.2 (A), J1.1 (Pin_1), J1.4 (Pin_4), J1.5 (Pin_5), J1.6 (Pin_6)
- net at U?.1 (GND): now also C4.2, C5.2, C6.2
- net at U?.2 (TR): now also U?.6 (THR), C6.1
- net at U?.4 (R): now also Q1.3 (D), R15.2
- net at U?.5 (CV): now also C4.1
- net at U?.7 (DIS): now also R16.2, R17.1
- net at U?.8 (VCC): now also C5.1, R15.1, R16.1
- new net: C3.2, D2.1 (K)
- new net: Q2.3 (D), R18.2
- new net: D3.1 (K), R19.1
- new net GRN+: J1.2 (Pin_2)
- new net RED+: D3.2 (A), J1.3 (Pin_3)
Other:
- moved on the sheet: U?
